File: CAD/V1.3.1/E-paper.kicad_sch (KiCad schematic)
At the start: 14 parts, among them K12 SFV33R-1STE9HLF, U12 E_D097OC1, U8 SN74LVC1G34DBV

Commit message: Updating open source files.
Parts:
- K12: value SFV33R-1STE9HLF -> SFV33R-1STBE1HLF
Changed lines of the file:
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@@
       (effects (font (size 1.27 1.27)) (justify left))
     )
-    (property "Value" "SFV33R-1STE9HLF" (id 1) (at 203.2 134.62 0)
+    (property "Value" "SFV33R-1STBE1HLF" (id 1) (at 203.2 134.62 0)
       (effects (font (size 1.27 1.27)) (justify left))
     )
