File: CAD/V1.3.1/SD_RTC_GPIO.kicad_sch (KiCad schematic)
At the start: 23 parts, among them K10 CR2032_BS-6-1, K11 HYC77-TF09-200, Q10 PMOS, SW3 K2-1114SA-A4SW-06, U7 PCF85063A, X1 7LC32768F12UC

Commit message: Updating open source files.
Parts:
- C34, C35: value DNP -> 12p
Changed lines of the file:
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@@
       (effects (font (size 1 1)) (justify right))
     )
-    (property "Value" "DNP" (id 1) (at 109.855 69.85 90)
+    (property "Value" "12p" (id 1) (at 109.855 69.85 90)
       (effects (font (size 1 1)) (justify right))
     )
@@
       (effects (font (size 1 1)) (justify right))
     )
-    (property "Value" "DNP" (id 1) (at 89.535 69.85 90)
+    (property "Value" "12p" (id 1) (at 89.535 69.85 90)
       (effects (font (size 1 1)) (justify right))
     )
